Commit message: Robot update

File: my_robot/urdf/my_robot.xacro (robot description, xacro)
@@ -1,6 +1,4 @@
 <robot name="my_robot" xmlns:xacro="http://www.ros.org/wiki/xacro">
-<xacro:include filename="$(find my_robot)/urdf/my_robot.gazebo" />
-  <link name="robot_footprint">
-  </link>
+  <link name="robot_footprint"></link>
   <joint name="robot_footprint_joint" type="fixed">
     <origin xyz="0 0 0" rpy="0 0 0" />
@@ -22,5 +20,5 @@
       <origin xyz="0 0 0" rpy=" 0 0 0"/>
       <geometry>
-        <box size=".4 .2 .1"/>
+        <box size=".5 .2 .1"/>
       </geometry>
     </collision>
@@ -28,5 +26,5 @@
       <origin xyz="0 0 0" rpy=" 0 0 0"/>
       <geometry>
-        <box size=".4 .2 .1"/>
+        <box size=".5 .2 .1"/>
       </geometry>
     </visual>
@@ -55,126 +53,135 @@
       </geometry>
     </visual>
+    <link name='rear_left_wheel'>
+      <pose>0 0 0.1 0 0 0</pose>
+      <inertial>
+        <mass value="5.0"/>
+        <origin xyz="0.0 0 0" rpy=" 0 1.5707 1.5707"/>
+        <inertia
+            ixx="0.1" ixy="0" ixz="0"
+            iyy="0.1" iyz="0"
+            izz="0.1"
+        />
+      </inertial>
+      <collision name='rear_left_wheel_collision'>
+        <origin xyz="0.0 0 0" rpy=" 0 1.5707 1.5707"/>
+        <geometry>
+          <cylinder radius="0.1" length="0.05"/>
+        </geometry>
+      </collision>
+      <visual name='rear_left_wheel'>
+        <origin xyz="0.0 0 0" rpy=" 0 1.5707 1.5707"/>
+        <geometry>
+          <cylinder radius="0.1" length="0.05"/>
+        </geometry>
+      </visual>
+    </link>
+    <joint type="continuous" name="rear_left_wheel_hinge">
+      <origin xyz="-0.125 -0.15 0" rpy="0 0 0"/>
+      <child link="rear_left_wheel"/>
+      <parent link="chassis"/>
+      <axis xyz="0 1 0" rpy="0 0 0"/>
+      <limit effort="10000" velocity="1000"/>
+      <dynamics damping="1.0" friction="1.0"/>
+    </joint>
+    <link name='front_left_wheel'>
+      <pose>0 0 0.1 0 0 0</pose>
+      <inertial>
+        <mass value="5.0"/>
+        <origin xyz="0.0 0 0" rpy=" 0 1.5707 1.5707"/>
+        <inertia
+            ixx="0.1" ixy="0" ixz="0"
+            iyy="0.1" iyz="0"
+            izz="0.1"
+        />
+      </inertial>
+      <collision name='front_left_wheel_collision'>
+        <origin xyz="0.0 0 0" rpy=" 0 1.5707 1.5707"/>
+        <geometry>
+          <cylinder radius="0.1" length="0.05"/>
+        </geometry>
+      </collision>
+      <visual name='front_left_wheel_visual'>
+        <origin xyz="0.0 0 0" rpy=" 0 1.5707 1.5707"/>
+        <geometry>
+          <cylinder radius="0.1" length="0.05"/>
+        </geometry>
+      </visual>
+    </link>
+    <joint type="continuous" name="front_left_wheel_hinge">
+      <origin xyz="0.125 -0.15 0" rpy="0 0 0"/>
+      <child link="front_left_wheel"/>
+      <parent link="chassis"/>
+      <axis xyz="0 1 0" rpy="0 0 0"/>
+      <limit effort="10000" velocity="1000"/>
+      <dynamics damping="1.0" friction="1.0"/>
+    </joint>
+    <link name='rear_right_wheel'>
+      <pose>0 0 0.1 0 0 0</pose>
+      <inertial>
+        <mass value="5.0"/>
+        <origin xyz="0.0 0 0" rpy=" 0 1.5707 1.5707"/>
+        <inertia
+            ixx="0.1" ixy="0" ixz="0"
+            iyy="0.1" iyz="0"
+            izz="0.1"
+        />
+      </inertial>
+      <collision name='rear_right_wheel_collision'>
+        <origin xyz="0.0 0 0" rpy=" 0 1.5707 1.5707"/>
+        <geometry>
+          <cylinder radius="0.1" length="0.05"/>
+        </geometry>
+      </collision>
+      <visual name='rear_right_wheel_visual'>
+        <origin xyz="0.0 0 0" rpy=" 0 1.5707 1.5707"/>
+        <geometry>
+          <cylinder radius="0.1" length="0.05"/>
+        </geometry>
+      </visual>
+    </link>
+    <joint type="continuous" name="rear_right_wheel_hinge">
+      <origin xyz="-0.125 0.15 0" rpy="0 0 0"/>
+      <child link="rear_right_wheel"/>
+      <parent link="chassis"/>
+      <axis xyz="0 1 0" rpy="0 0 0"/>
+      <limit effort="10000" velocity="1000"/>
+      <dynamics damping="1.0" friction="1.0"/>
+    </joint>
+    <link name='front_right_wheel'>
+      <pose>0 0 0.1 0 0 0</pose>
+      <inertial>
+        <mass value="5.0"/>
+        <origin xyz="0.0 0 0" rpy=" 0 1.5707 1.5707"/>
+        <inertia
+            ixx="0.1" ixy="0" ixz="0"
+            iyy="0.1" iyz="0"
+            izz="0.1"
+        />
+      </inertial>
+      <collision name='front_right_wheel_collision'>
+        <origin xyz="0.0 0 0" rpy=" 0 1.5707 1.5707"/>
+        <geometry>
+          <cylinder radius="0.1" length="0.05"/>
+        </geometry>
+      </collision>
+      <visual name='front_right_wheel_visual'>
+        <origin xyz="0.0 0 0" rpy=" 0 1.5707 1.5707"/>
+        <geometry>
+          <cylinder radius="0.1" length="0.05"/>
+        </geometry>
+      </visual>
+    </link>
+    <joint type="continuous" name="front_right_wheel_hinge">
+      <origin xyz="0.125 0.15 0" rpy="0 0 0"/>
+      <child link="front_right_wheel"/>
+      <parent link="chassis"/>
+      <axis xyz="0 1 0" rpy="0 0 0"/>
+      <limit effort="10000" velocity="1000"/>
+      <dynamics damping="1.0" friction="1.0"/>
+    </joint>
   </link>
-  <link name='left_wheel'>
-    <pose>0 0 0.1 0 0 0</pose>
-    <inertial>
-      <mass value="5.0"/>
-      <origin xyz="0.0 0 0" rpy=" 0 1.5707 1.5707"/>
-      <inertia
-          ixx="0.1" ixy="0" ixz="0"
-          iyy="0.1" iyz="0"
-          izz="0.1"
-      />
-    </inertial>
-    <collision name='left_wheel_collision'>
-      <origin xyz="0.0 0 0" rpy=" 0 1.5707 1.5707"/>
-      <geometry>
-        <cylinder radius="0.1" length="0.05"/>
-      </geometry>
-    </collision>
-    <visual name='left_wheel_visual'>
-      <origin xyz="0.0 0 0" rpy=" 0 1.5707 1.5707"/>
-      <geometry>
-        <cylinder radius="0.1" length="0.05"/>
-      </geometry>
-    </visual>
-  </link>
-  <joint type="continuous" name="left_wheel_hinge">
-    <origin xyz="0 -0.15 0" rpy="0 0 0"/>
-    <child link="left_wheel"/>
-    <parent link="chassis"/>
-    <axis xyz="0 1 0" rpy="0 0 0"/>
-    <limit effort="10000" velocity="1000"/>
-    <dynamics damping="1.0" friction="1.0"/>
-  </joint>
-  <link name='right_wheel'>
-    <pose>0 0 0.1 0 0 0</pose>
-    <inertial>
-      <mass value="5.0"/>
-      <origin xyz="0.0 0 0" rpy=" 0 1.5707 1.5707"/>
-      <inertia
-          ixx="0.1" ixy="0" ixz="0"
-          iyy="0.1" iyz="0"
-          izz="0.1"
-      />
-    </inertial>
-    <collision name='right_wheel_collision'>
-      <origin xyz="0.0 0 0" rpy=" 0 1.5707 1.5707"/>
-      <geometry>
-        <cylinder radius="0.1" length="0.05"/>
-      </geometry>
-    </collision>
-    <visual name='right_wheel_visual'>
-      <origin xyz="0.0 0 0" rpy=" 0 1.5707 1.5707"/>
-      <geometry>
-        <cylinder radius="0.1" length="0.05"/>
-      </geometry>
-    </visual>
-  </link>
-  <joint type="continuous" name="right_wheel_hinge">
-    <origin xyz="0 0.15 0" rpy="0 0 0"/>
-    <child link="right_wheel"/>
-    <parent link="chassis"/>
-    <axis xyz="0 1 0" rpy="0 0 0"/>
-    <limit effort="10000" velocity="1000"/>
-    <dynamics damping="1.0" friction="1.0"/>
-  </joint>
-  <link name='camera'>
-    <inertial>
-      <mass value="0.1"/>
-      <origin xyz="0.0 0 0" rpy=" 0 0 0"/>
-      <inertia
-          ixx="1e-6" ixy="0" ixz="0"
-          iyy="1e-6" iyz="0"
-          izz="1e-6"
-      />
-    </inertial>
-    <collision name='camera_collision'>
-      <origin xyz="0.0 0 0" rpy=" 0 0 0"/>
-      <geometry>
-        <box size="0.05 0.05 0.05"/>
-      </geometry>
-    </collision>
-    <visual name='camera_visual'>
-      <origin xyz="0.0 0 0" rpy=" 0 0 0"/>
-      <geometry>
-        <box size="0.05 0.05 0.05"/>
-      </geometry>
-    </visual>
-  </link>
-  <joint type="fixed" name="camera_joint">
-    <origin xyz="0.2 0 0" rpy="0 0 0"/>
-    <child link="camera"/>
-    <parent link="chassis"/>
-    <axis xyz="0 1 0" rpy="0 0 0"/>
-  </joint>
-  <link name='hokuyo'>
-    <inertial>
-      <mass value="1e-5"/>
-      <origin xyz="0.0 0 0" rpy=" 0 0 0"/>
-      <inertia
-          ixx="1e-6" ixy="0" ixz="0"
-          iyy="1e-6" iyz="0"
-          izz="1e-6"
-      />
-    </inertial>
-    <collision name='hokuyo_collision'>
-      <origin xyz="0.0 0 0" rpy=" 0 0 0"/>
-      <geometry>
-        <box size="0.1 0.1 0.1"/>
-      </geometry>
-    </collision>
-    <visual name='hokuyo_visual'>
-      <origin xyz="0.0 0 0" rpy=" 0 0 0"/>
-      <geometry>
-        <mesh filename ="package://my_robot/meshes/hokuyo.dae"/>
-      </geometry>
-    </visual>
-  </link>
-  <joint type="fixed" name="hokuyo_joint">
-    <origin xyz="0.15 0 .1" rpy="0 0 0"/>
-    <child link="hokuyo"/>
-    <parent link="chassis"/>
-    <axis xyz="0 1 0" rpy="0 0 0"/>
-  </joint>
+  <gazebo reference="chassis">
+    <material>Gazebo/Orange</material>
+  </gazebo>
 </robot>

Commit message: resubmission

File: my_robot/urdf/my_robot.xacro (robot description, xacro)
@@ -1,3 +1,4 @@
 <robot name="my_robot" xmlns:xacro="http://www.ros.org/wiki/xacro">
+<xacro:include filename="$(find my_robot)/urdf/my_robot.gazebo" />
   <link name="robot_footprint"></link>
   <joint name="robot_footprint_joint" type="fixed">
@@ -20,5 +21,5 @@
       <origin xyz="0 0 0" rpy=" 0 0 0"/>
       <geometry>
-        <box size=".5 .2 .1"/>
+        <box size=".5 .2 0.1075"/>
       </geometry>
     </collision>
@@ -26,32 +27,9 @@
       <origin xyz="0 0 0" rpy=" 0 0 0"/>
       <geometry>
-        <box size=".5 .2 .1"/>
+        <box size=".5 .2 0.1075"/>
       </geometry>
     </visual>
-    <collision name='back_caster_collision'>
-      <origin xyz="-0.15 0 -0.05" rpy=" 0 0 0"/>
-      <geometry>
-        <sphere radius="0.0499"/>
-      </geometry>
-    </collision>
-    <visual name='back_caster_visual'>
-      <origin xyz="-0.15 0 -0.05" rpy=" 0 0 0"/>
-      <geometry>
-        <sphere radius="0.05"/>
-      </geometry>
-    </visual>
-    <collision name='front_caster_collision'>
-      <origin xyz="0.15 0 -0.05" rpy=" 0 0 0"/>
-      <geometry>
-        <sphere radius="0.0499"/>
-      </geometry>
-    </collision>
-    <visual name='front_caster_visual'>
-      <origin xyz="0.15 0 -0.05" rpy=" 0 0 0"/>
-      <geometry>
-        <sphere radius="0.05"/>
-      </geometry>
-    </visual>
-    <link name='rear_left_wheel'>
+  </link>
+  <link name='rear_left_wheel'>
       <pose>0 0 0.1 0 0 0</pose>
       <inertial>
@@ -67,5 +45,5 @@
         <origin xyz="0.0 0 0" rpy=" 0 1.5707 1.5707"/>
         <geometry>
-          <cylinder radius="0.1" length="0.05"/>
+          <cylinder radius="0.1075" length="0.05"/>
         </geometry>
       </collision>
@@ -73,9 +51,9 @@
         <origin xyz="0.0 0 0" rpy=" 0 1.5707 1.5707"/>
         <geometry>
-          <cylinder radius="0.1" length="0.05"/>
-        </geometry>
-      </visual>
-    </link>
-    <joint type="continuous" name="rear_left_wheel_hinge">
+          <cylinder radius="0.1075" length="0.05"/>
+        </geometry>
+      </visual>
+  </link>
+  <joint type="continuous" name="rear_left_wheel_hinge">
       <origin xyz="-0.125 -0.15 0" rpy="0 0 0"/>
       <child link="rear_left_wheel"/>
@@ -84,6 +62,6 @@
       <limit effort="10000" velocity="1000"/>
       <dynamics damping="1.0" friction="1.0"/>
-    </joint>
-    <link name='front_left_wheel'>
+  </joint>
+  <link name='front_left_wheel'>
       <pose>0 0 0.1 0 0 0</pose>
       <inertial>
@@ -99,5 +77,5 @@
         <origin xyz="0.0 0 0" rpy=" 0 1.5707 1.5707"/>
         <geometry>
-          <cylinder radius="0.1" length="0.05"/>
+          <cylinder radius="0.1075" length="0.05"/>
         </geometry>
       </collision>
@@ -105,8 +83,8 @@
         <origin xyz="0.0 0 0" rpy=" 0 1.5707 1.5707"/>
         <geometry>
-          <cylinder radius="0.1" length="0.05"/>
-        </geometry>
-      </visual>
-    </link>
+          <cylinder radius="0.1075" length="0.05"/>
+        </geometry>
+      </visual>
+  </link>
     <joint type="continuous" name="front_left_wheel_hinge">
       <origin xyz="0.125 -0.15 0" rpy="0 0 0"/>
@@ -117,5 +95,5 @@
       <dynamics damping="1.0" friction="1.0"/>
     </joint>
-    <link name='rear_right_wheel'>
+  <link name='rear_right_wheel'>
       <pose>0 0 0.1 0 0 0</pose>
       <inertial>
@@ -131,5 +109,5 @@
         <origin xyz="0.0 0 0" rpy=" 0 1.5707 1.5707"/>
         <geometry>
-          <cylinder radius="0.1" length="0.05"/>
+          <cylinder radius="0.1075" length="0.05"/>
         </geometry>
       </collision>
@@ -137,8 +115,8 @@
         <origin xyz="0.0 0 0" rpy=" 0 1.5707 1.5707"/>
         <geometry>
-          <cylinder radius="0.1" length="0.05"/>
-        </geometry>
-      </visual>
-    </link>
+          <cylinder radius="0.1075" length="0.05"/>
+        </geometry>
+      </visual>
+  </link>
     <joint type="continuous" name="rear_right_wheel_hinge">
       <origin xyz="-0.125 0.15 0" rpy="0 0 0"/>
@@ -149,5 +127,5 @@
       <dynamics damping="1.0" friction="1.0"/>
     </joint>
-    <link name='front_right_wheel'>
+  <link name='front_right_wheel'>
       <pose>0 0 0.1 0 0 0</pose>
       <inertial>
@@ -163,5 +141,5 @@
         <origin xyz="0.0 0 0" rpy=" 0 1.5707 1.5707"/>
         <geometry>
-          <cylinder radius="0.1" length="0.05"/>
+          <cylinder radius="0.1075" length="0.05"/>
         </geometry>
       </collision>
@@ -169,8 +147,8 @@
         <origin xyz="0.0 0 0" rpy=" 0 1.5707 1.5707"/>
         <geometry>
-          <cylinder radius="0.1" length="0.05"/>
-        </geometry>
-      </visual>
-    </link>
+          <cylinder radius="0.1075" length="0.05"/>
+        </geometry>
+      </visual>
+  </link>
     <joint type="continuous" name="front_right_wheel_hinge">
       <origin xyz="0.125 0.15 0" rpy="0 0 0"/>
@@ -181,7 +159,76 @@
       <dynamics damping="1.0" friction="1.0"/>
     </joint>
-  </link>
   <gazebo reference="chassis">
     <material>Gazebo/Orange</material>
   </gazebo>
+  <gazebo reference="rear_left_wheel">
+    <material>Gazebo/Green</material>
+  </gazebo>
+  <gazebo reference="front_left_wheel">
+    <material>Gazebo/Green</material>
+  </gazebo>
+  <gazebo reference="rear_right_wheel">
+    <material>Gazebo/Green</material>
+  </gazebo>
+  <gazebo reference="front_right_wheel">
+    <material>Gazebo/Green</material>
+  </gazebo>
+  <link name='camera'>
+    <inertial>
+      <mass value="0.1"/>
+      <origin xyz="0.0 0 0" rpy=" 0 0 0"/>
+      <inertia
+          ixx="1e-6" ixy="0" ixz="0"
+          iyy="1e-6" iyz="0"
+          izz="1e-6"
+      />
+    </inertial>
+    <collision name='camera_collision'>
+      <origin xyz="0.0 0 0" rpy=" 0 0 0"/>
+      <geometry>
+        <box size="0.05 0.05 0.05"/>
+      </geometry>
+    </collision>
+    <visual name='camera_visual'>
+      <origin xyz="0.0 0 0" rpy=" 0 0 0"/>
+      <geometry>
+        <box size="0.05 0.05 0.05"/>
+      </geometry>
+    </visual>
+  </link>
+  <joint type="fixed" name="camera_joint">
+    <origin xyz="0.25 0 0" rpy="0 0 0"/>
+    <child link="camera"/>
+    <parent link="chassis"/>
+    <axis xyz="0 1 0" rpy="0 0 0"/>
+  </joint>
+  <link name='hokuyo'>
+    <inertial>
+      <mass value="1e-5"/>
+      <origin xyz="0.0 0 0" rpy=" 0 0 0"/>
+      <inertia
+          ixx="1e-6" ixy="0" ixz="0"
+          iyy="1e-6" iyz="0"
+          izz="1e-6"
+      />
+    </inertial>
+    <collision name='hokuyo_collision'>
+      <origin xyz="0.0 0 0" rpy=" 0 0 0"/>
+      <geometry>
+        <box size="0.1 0.1 0.1"/>
+      </geometry>
+    </collision>
+    <visual name='hokuyo_visual'>
+      <origin xyz="0.0 0 0" rpy=" 0 0 0"/>
+      <geometry>
+        <mesh filename ="package://my_robot/meshes/hokuyo.dae"/>
+      </geometry>
+    </visual>
+  </link>
+  <joint type="fixed" name="hokuyo_joint">
+    <origin xyz="0.15 0 0.1075" rpy="0 0 0"/>
+    <child link="hokuyo"/>
+    <parent link="chassis"/>
+    <axis xyz="0 1 0" rpy="0 0 0"/>
+  </joint>
 </robot>

Commit message: commit2

File: my_robot/urdf/my_robot.xacro (robot description, xacro)
@@ -8,5 +8,5 @@
   </joint>
   <link name='chassis'>
-    <pose>0 0 0.1 0 0 0</pose>
+    <pose>0 0 0.1075 0 0 0</pose>
     <inertial>
       <mass value="15.0"/>
@@ -32,5 +32,5 @@
   </link>
   <link name='rear_left_wheel'>
-      <pose>0 0 0.1 0 0 0</pose>
+      <pose>0 0 0.1075 0 0 0</pose>
       <inertial>
         <mass value="5.0"/>
@@ -56,5 +56,5 @@
   </link>
   <joint type="continuous" name="rear_left_wheel_hinge">
-      <origin xyz="-0.125 -0.15 0" rpy="0 0 0"/>
+      <origin xyz="-0.126 -0.126 0" rpy="0 0 0"/>
       <child link="rear_left_wheel"/>
       <parent link="chassis"/>
@@ -64,5 +64,5 @@
   </joint>
   <link name='front_left_wheel'>
-      <pose>0 0 0.1 0 0 0</pose>
+      <pose>0 0 0.1075 0 0 0</pose>
       <inertial>
         <mass value="5.0"/>
@@ -88,5 +88,5 @@
   </link>
     <joint type="continuous" name="front_left_wheel_hinge">
-      <origin xyz="0.125 -0.15 0" rpy="0 0 0"/>
+      <origin xyz="0.126 -0.126 0" rpy="0 0 0"/>
       <child link="front_left_wheel"/>
       <parent link="chassis"/>
@@ -96,5 +96,5 @@
     </joint>
   <link name='rear_right_wheel'>
-      <pose>0 0 0.1 0 0 0</pose>
+      <pose>0 0 0.1075 0 0 0</pose>
       <inertial>
         <mass value="5.0"/>
@@ -120,5 +120,5 @@
   </link>
     <joint type="continuous" name="rear_right_wheel_hinge">
-      <origin xyz="-0.125 0.15 0" rpy="0 0 0"/>
+      <origin xyz="-0.126 0.126 0" rpy="0 0 0"/>
       <child link="rear_right_wheel"/>
       <parent link="chassis"/>
@@ -128,5 +128,5 @@
     </joint>
   <link name='front_right_wheel'>
-      <pose>0 0 0.1 0 0 0</pose>
+      <pose>0 0 0.1075 0 0 0</pose>
       <inertial>
         <mass value="5.0"/>
@@ -152,5 +152,5 @@
   </link>
     <joint type="continuous" name="front_right_wheel_hinge">
-      <origin xyz="0.125 0.15 0" rpy="0 0 0"/>
+      <origin xyz="0.126 0.126 0" rpy="0 0 0"/>
       <child link="front_right_wheel"/>
       <parent link="chassis"/>
@@ -232,3 +232,10 @@
     <axis xyz="0 1 0" rpy="0 0 0"/>
   </joint>
+  <link name="camera_link_optical">
+  </link>
+  <joint name="camera_optical_joint" type="fixed">
+    <origin xyz="0 0 0" rpy="-1.5707 0 -1.5707"/>
+    <parent link="camera"/>
+    <child link="camera_link_optical"/>
+  </joint>
 </robot>
